Commit message: One more link added to the robot arm and robot arm created in a different robot

File: my_robot_description/urdf/arm.xacro (robot description, xacro)
@@ -20,5 +20,5 @@
             <origin xyz="0 0 0" rpy="0 0 0" />
         </collision>
-        <xacro:box_inertia m="1.0" x="${arm_base_length}" y="${arm_base_width}" z="${arm_base_height}"
+        <xacro:box_inertia m="500.0" x="${arm_base_length}" y="${arm_base_width}" z="${arm_base_height}"
                            o_xyz="0 0 0" o_rpy="0 0 0" />
     </link>
@@ -40,14 +40,38 @@
                                 o_xyz="0 0 ${forearm_length/2}" o_rpy="0 0 0" />
     </link>
-    <joint name="arm_base_joint" type="fixed">
+    <link name="wrist_link">
+        <visual>
+            <geometry>
+                <cylinder radius="${forearm_radius}" length="${forearm_length}" />
+            </geometry>
+            <origin xyz="0 0 ${forearm_length/2}" rpy="0 0 0" />
+            <material name="orange" />
+        </visual>
+        <collision>
+            <geometry>
+                <cylinder radius="${forearm_radius}" length="${forearm_length}" />
+            </geometry>
+            <origin xyz="0 0 ${forearm_length/2}" rpy="0 0 0" />
+        </collision>
+        <xacro:cylinder_inertia m="1.0" r="${forearm_radius}" l="${forearm_length}"
+                                o_xyz="0 0 ${forearm_length/2}" o_rpy="0 0 0" />
+    </link>
+    <!--joint name="arm_base_joint" type="fixed">
         <parent link="base_link" />
         <child link="arm_base_link" />
         <origin xyz="${base_length/4} 0 ${base_height}" rpy="0 0 0"/>
-    </joint>
+    </joint> -->
     <joint name="forearm_arm_base_joint" type="revolute">
         <parent link="arm_base_link" />
         <child link="forearm_link" />
         <origin xyz="0 0 0" rpy="0 0 0" />
-        <limit effort="1000.0" lower="0.0" upper="1" velocity="0.5"/>
+        <limit effort="1000.0" lower="-1.57" upper="1.57" velocity="0.5"/>
+        <axis xyz="0 1 0" />
+    </joint>
+    <joint name="forearm_wrist_joint" type="revolute">
+        <parent link="forearm_link" />
+        <child link="wrist_link" />
+        <origin xyz="0 0 ${forearm_length}" rpy="0 0 0" />
+        <limit effort="1000.0" lower="-1.57" upper="1.57" velocity="0.5"/>
         <axis xyz="0 1 0" />
     </joint>

Commit message: combined both robots

File: my_robot_description/urdf/arm.xacro (robot description, xacro)
@@ -57,9 +57,9 @@
                                 o_xyz="0 0 ${forearm_length/2}" o_rpy="0 0 0" />
     </link>
-    <!--joint name="arm_base_joint" type="fixed">
+    <joint name="arm_base_joint" type="fixed">
         <parent link="base_link" />
         <child link="arm_base_link" />
         <origin xyz="${base_length/4} 0 ${base_height}" rpy="0 0 0"/>
-    </joint> -->
+    </joint>
     <joint name="forearm_arm_base_joint" type="revolute">
         <parent link="arm_base_link" />

File: my_robot_description/urdf/my_robot.urdf.xacro (robot description, xacro)
@@ -6,3 +6,4 @@
     <xacro:include filename="camera.xacro" />
     <xacro:include filename="arm.xacro"/>
+    <xacro:include filename="arm_gazebo.xacro"/>
 </robot>
